File: kicad-project/pixie-e.kicad_pcb (KiCad board)
At the start: 2 copper layers, 55 x 50 mm, 54 parts, among them J1 PWR, J2 ANT, J3 SP, J4 KEY, Q1 9018, Q2 2N2222, Q3 2N2222, Q4 2N3906, Q5 2N7000, SW1 PWR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

Commit message: Change Q1 to 2N2222.
Parts:
- Q1: value 9018 -> 2N2222
Changed lines of the file:
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@@
     (add_net "Net-(Q5-Pad2)")
     (add_net "Net-(R8-Pad2)")
+    (add_net "Net-(U1-Pad7)")
     (add_net Phone)
     (add_net SHIFT)
@@
       (effects (font (size 1 1) (thickness 0.15)))
     )
-    (fp_text value 9018 (at 2.54 2.79 90) (layer F.Fab)
+    (fp_text value 2N2222 (at 2.54 2.79 90) (layer F.Fab)
       (effects (font (size 1 1) (thickness 0.15)))
     )
@@
   (segment (start 136.799999 85.799999) (end 138 87) (width 0.25) (layer F.Cu) (net 8))
   (segment (start 131.5 85) (end 132.299999 85.799999) (width 0.25) (layer F.Cu) (net 8))
+  (segment (start 145.304821 94) (end 145.504821 93.8) (width 0.25) (layer F.Cu) (net 8))
+  (segment (start 138.5 94) (end 145.304821 94) (width 0.25) (layer F.Cu) (net 8))
   (segment (start 147.04 60) (end 150.2 60) (width 0.25) (layer F.Cu) (net 9))
   (segment (start 144.04 57) (end 147.04 60) (width 0.25) (layer F.Cu) (net 9))
@@
   (segment (start 125.5 70.5) (end 122.665001 73.334999) (width 0.25) (layer B.Cu) (net 11))
   (segment (start 125.5 69.5) (end 125.5 70.5) (width 0.25) (layer B.Cu) (net 11))
+  (segment (start 119 94.1) (end 119.4 94.5) (width 0.25) (layer F.Cu) (net 11))
+  (segment (start 119 90) (end 119 94.1) (width 0.25) (layer F.Cu) (net 11))
   (segment (start 139.884821 75.08) (end 139.75137 75.08) (width 0.25) (layer B.Cu) (net 12))
   (segment (start 144.604821 79.8) (end 139.884821 75.08) (width 0.25) (layer B.Cu) (net 12))
@@
   (segment (start 135.636 71.824315) (end 133.811685 70) (width 0.25) (layer F.Cu) (net 14))
   (segment (start 135.636 72.39) (end 135.636 71.824315) (width 0.25) (layer F.Cu) (net 14))
+  (segment (start 135.5 92) (end 137.535001 89.964999) (width 0.25) (layer B.Cu) (net 14))
+  (segment (start 135.636 79.170998) (end 135.636 72.39) (width 0.25) (layer B.Cu) (net 14))
+  (segment (start 137.535001 89.964999) (end 137.535001 82.930001) (width 0.25) (layer B.Cu) (net 14))
+  (segment (start 137.877001 81.411999) (end 135.636 79.170998) (width 0.25) (layer B.Cu) (net 14))
+  (segment (start 137.535001 82.930001) (end 137.877001 82.588001) (width 0.25) (layer B.Cu) (net 14))
+  (segment (start 137.877001 82.588001) (end 137.877001 81.411999) (width 0.25) (layer B.Cu) (net 14))
+  (segment (start 135.5 92) (end 129 92) (width 0.25) (layer B.Cu) (net 14))
   (segment (start 131.240001 67.299999) (end 132.04 66.5) (width 0.25) (layer F.Cu) (net 15))
   (segment (start 127.249999 71.290001) (end 131.240001 67.299999) (width 0.25) (layer F.Cu) (net 15))
@@
   (segment (start 102.87 87.87) (end 103 88) (width 0.25) (layer F.Cu) (net 18))
   (segment (start 102.87 84.836) (end 102.87 87.87) (width 0.25) (layer F.Cu) (net 18))
-  (segment (start 145.304821 94) (end 145.504821 93.8) (width 0.25) (layer F.Cu) (net 8))
-  (segment (start 138.5 94) (end 145.304821 94) (width 0.25) (layer F.Cu) (net 8))
-  (segment (start 119 94.1) (end 119.4 94.5) (width 0.25) (layer F.Cu) (net 11))
-  (segment (start 119 90) (end 119 94.1) (width 0.25) (layer F.Cu) (net 11))
-  (segment (start 135.5 92) (end 137.535001 89.964999) (width 0.25) (layer B.Cu) (net 14))
-  (segment (start 135.636 79.170998) (end 135.636 72.39) (width 0.25) (layer B.Cu) (net 14))
-  (segment (start 137.535001 89.964999) (end 137.535001 82.930001) (width 0.25) (layer B.Cu) (net 14))
-  (segment (start 137.877001 81.411999) (end 135.636 79.170998) (width 0.25) (layer B.Cu) (net 14))
-  (segment (start 137.535001 82.930001) (end 137.877001 82.588001) (width 0.25) (layer B.Cu) (net 14))
-  (segment (start 137.877001 82.588001) (end 137.877001 81.411999) (width 0.25) (layer B.Cu) (net 14))
-  (segment (start 135.5 92) (end 129 92) (width 0.25) (layer B.Cu) (net 14))
   (segment (start 107.5 94.5) (end 108.45 94.5) (width 0.25) (layer F.Cu) (net 19))
   (segment (start 119.174999 97.225001) (end 121.4 95) (width 0.25) (layer F.Cu) (net 19))
